File: Z80Computer.kicad_pcb (KiCad board)
At the start: 2 copper layers, 154.9 x 129.5 mm, 13 parts, among them J1 Conn_Coaxial_Power, SW1 SW_Push, U1 Z80CPU, U2 28C256, U4 74LS138, U5 74LS00, U6 KM62256CLP, U7 74LS00, X1 CXO_DIP14

Commit message: before auto route pcb
Parts:
- removed the U2 at (96.5, 119.4)
- added C1: 0.1uF, Capacitor_THT:CP_Radial_D4.0mm_P1.50mm, F.Cu at (90.4, 78.7)
- added C2: 0.1uF, Capacitor_THT:CP_Radial_D4.0mm_P1.50mm, F.Cu at (99.1, 78.7)
- added D1: 1N4148, Diode_THT:D_DO-35_SOD27_P7.62mm_Horizontal, F.Cu at (176.5, 81.3)
- added D2: 1N4148, Diode_THT:D_DO-35_SOD27_P7.62mm_Horizontal, F.Cu at (184.2, 86.4)
- added D3: 1N4148, Diode_THT:D_DO-35_SOD27_P7.62mm_Horizontal, F.Cu at (184.2, 91.4)
- added D4: 1N4148, Diode_THT:D_DO-35_SOD27_P7.62mm_Horizontal, F.Cu at (184.2, 96.5)
- added D5: 1N4148, Diode_THT:D_DO-35_SOD27_P7.62mm_Horizontal, F.Cu at (184.2, 101.6)
- added D6: 1N4148, Diode_THT:D_DO-35_SOD27_P7.62mm_Horizontal, F.Cu at (184.2, 106.7)
- added D7: 1N4148, Diode_THT:D_DO-35_SOD27_P7.62mm_Horizontal, F.Cu at (184.2, 111.8)
- added D8: 1N4148, Diode_THT:D_DO-35_SOD27_P7.62mm_Horizontal, F.Cu at (184.2, 116.8)
- added D9: LED, LED_THT:LED_D5.0mm, F.Cu at (55.9, 50.8)
- added IC2_EEPROM1: 28C256, Package_DIP:DIP-28_W15.24mm, F.Cu at (94.0, 125.7)
- added IC6_SRAM1: KM62256CLP, Package_DIP:DIP-28_W15.24mm, F.Cu at (121.9, 125.7)
- added J2: Conn_01x08_Pin, Connector_JST:JST_EH_B8B-EH-A_1x08_P2.50mm_Vertical, F.Cu at (193.6, 132.1)
- added J3: Conn_01x08_Pin, Connector_JST:JST_EH_B8B-EH-A_1x08_P2.50mm_Vertical, F.Cu at (193.0, 109.0)
- added R1: 1K, Resistor_THT:R_Axial_DIN0204_L3.6mm_D1.6mm_P1.90mm_Vertical, F.Cu at (66.7, 40.6)
- added R10: 440R, Resistor_THT:R_Axial_DIN0204_L3.6mm_D1.6mm_P1.90mm_Vertical, F.Cu at (61.6, 50.8)
- added R3: 10K, Resistor_THT:R_Axial_DIN0204_L3.6mm_D1.6mm_P1.90mm_Vertical, F.Cu at (176.5, 148.0)
- added R4: 10K, Resistor_THT:R_Axial_DIN0204_L3.6mm_D1.6mm_P1.90mm_Vertical, F.Cu at (176.5, 152.8)
- added R5: 10K, Resistor_THT:R_Axial_DIN0204_L3.6mm_D1.6mm_P1.90mm_Vertical, F.Cu at (176.5, 143.3)
- added R6: 10K, Resistor_THT:R_Axial_DIN0204_L3.6mm_D1.6mm_P1.90mm_Vertical, F.Cu at (176.5, 138.6)
- added R7: 10K, Resistor_THT:R_Axial_DIN0204_L3.6mm_D1.6mm_P1.90mm_Vertical, F.Cu at (176.5, 133.9)
- added R8: 10K, Resistor_THT:R_Axial_DIN0204_L3.6mm_D1.6mm_P1.90mm_Vertical, F.Cu at (176.5, 129.2)
- added R9: 10K, Resistor_THT:R_Axial_DIN0204_L3.6mm_D1.6mm_P1.90mm_Vertical, F.Cu at (176.5, 124.5)
- added U3: 74LS273, Package_DIP:DIP-20_W7.62mm, F.Cu at (111.8, 83.8)
- added U7: 74LS00, Package_DIP:DIP-14_W7.62mm, F.Cu at (157.5, 99.0)
- R2: renamed from R1; value R_Small -> 10K
- U1: renamed from U7; value 74LS00 -> 74LS244; footprint Package_DIP:DIP-14_W7.62mm -> Package_DIP:DIP-20_W7.62mm
- U2: renamed from U5; value 74LS00 -> 74LS32
- U5: renamed from U3; value ~ -> 74LS00; footprint TestPoint:TestPoint_2Pads_Pitch2.54mm_Drill0.8mm -> Package_DIP:DIP-14_W7.62mm
- U6: value KM62256CLP -> 74LS244; footprint Package_DIP:DIP-28_W15.24mm -> Package_DIP:DIP-20_W7.62mm
- moved X1 122.0 mm to (61.0, 96.5)
- moved DIS1 71.4 mm to (157.9, 70.9), turned to 180 degrees
- moved U1 69.6 mm to (124.5, 91.4)
- moved SW1 52.6 mm to (167.6, 57.1)
- moved R2 45.7 mm to (176.5, 157.5)
- moved U5 41.9 mm to (141.0, 99.0)
- moved RV1 29.0 mm to (152.4, 78.7)
- moved U6 25.0 mm to (157.5, 129.5)
- moved U4 17.3 mm to (108.0, 96.5)
- moved U2 10.8 mm to (91.4, 99.0)
- moved IC1 6.36 mm to (55.9, 110.5)
- renumbered U1 to IC1
Connections:
- DIS1 pad P$1: GND -> Z80_PWRCAP
- DIS1 pad P$16: GND -> Z80_PWRCAP
- IC1 pad 26: Net-(U1-~{RESET}) -> Net-(IC1-~{RESET})
- IC1 pad 29: GND -> Z80_PWRCAP
- J1 pad 2: GND -> Z80_PWRCAP
- R2 pad 1: +5V -> Net-(J2-Pin_8)
- R2 pad 2: Net-(U1-~{RESET}) -> Z80_PWRCAP
- RV1 pad 3: GND -> Z80_PWRCAP
- SW1 pad 1: GND -> Z80_PWRCAP
- SW1 pad 2: Net-(U1-~{RESET}) -> Net-(IC1-~{RESET})
- U1 pad 1: /A15 -> Net-(U1-OEa)
- U1 pad 10: unconnected-(U7-Pad10) -> Z80_PWRCAP
- U1 pad 11: unconnected-(U7-Pad11) -> /D4
- U1 pad 12: unconnected-(U7-Pad12) -> Net-(J2-Pin_4)
- U1 pad 13: unconnected-(U7-Pad13) -> /D5
- U1 pad 14: +5V -> Net-(J2-Pin_3)
- U1 pad 2: ~{MREQ} -> /D0
- U1 pad 3: Net-(U2-~{CS}) -> Net-(J2-Pin_8)
- U1 pad 4: /A15 -> /D1
- U1 pad 5: /A15 -> Net-(J2-Pin_7)
- U1 pad 6: Net-(U5-Pad9) -> /D2
- U1 pad 7: GND -> Net-(J2-Pin_6)
- U1 pad 8: unconnected-(U7-Pad8) -> /D3
- U1 pad 9: unconnected-(U7-Pad9) -> Net-(J2-Pin_5)
- U2 pad 1: ~{RD} -> ~{KEYPAD_PORT}
- U2 pad 10: ~{MREQ} -> unconnected-(U2-Pad10)
- U2 pad 3: Net-(DIS1-PadP$5) -> Net-(U1-OEa)
- U2 pad 4: Net-(U4-O0) -> ~{WR}
- U2 pad 5: Net-(U4-O0) -> ~{KEYPAD_PORT}
- U2 pad 6: Net-(DIS1-PadP$6) -> Net-(U3-Cp)
- U2 pad 7: GND -> Z80_PWRCAP
- U2 pad 8: Net-(U6-~{CS}) -> unconnected-(U2-Pad8)
- U2 pad 9: Net-(U5-Pad9) -> unconnected-(U2-Pad9)
- U4 pad 14: unconnected-(U4-O1-Pad14) -> ~{KEYPAD_PORT}
- U4 pad 15: Net-(U4-O0) -> ~{LCD_OUT_PORT}
- U4 pad 8: GND -> Z80_PWRCAP
- U5 pad 1: (no net) -> ~{RD}
- U5 pad 2: (no net) -> ~{RD}
- U6 pad 1: /A14 -> Net-(U1-OEa)
- U6 pad 10: /A0 -> Z80_PWRCAP
- U6 pad 11: /D0 -> /D4
- U6 pad 12: /D1 -> Net-(J2-Pin_4)
- U6 pad 13: /D2 -> /D5
- U6 pad 14: GND -> Net-(J2-Pin_3)
- U6 pad 15: /D3 -> /D6
- U6 pad 16: /D4 -> Net-(J2-Pin_2)
- U6 pad 17: /D5 -> /D7
- U6 pad 18: /D6 -> Net-(J2-Pin_1)
- U6 pad 19: /D7 -> Net-(U1-OEa)
- U6 pad 2: /A12 -> /D0
- U6 pad 20: Net-(U6-~{CS}) -> +5V
- U6 pad 3: /A7 -> Net-(J2-Pin_8)
- U6 pad 4: /A6 -> /D1
- U6 pad 5: /A5 -> Net-(J2-Pin_7)
- U6 pad 6: /A4 -> /D2
- U6 pad 7: /A3 -> Net-(J2-Pin_6)
- U6 pad 8: /A2 -> /D3
- U6 pad 9: /A1 -> Net-(J2-Pin_5)
- X1 pad 7: GND -> Z80_PWRCAP
Routing:
- net GND: track 426.9 -> 0.00 mm
- net +5V: track 419.3 -> 0.00 mm
- net /D3: track 223.1 -> 0.00 mm, vias 1 -> 0
- net /D5: track 221.7 -> 0.00 mm
- net /D6: track 220.7 -> 0.00 mm
- net /D4: track 218.1 -> 0.00 mm, vias 1 -> 0
- net /D2: track 203.3 -> 0.00 mm
- net /D7: track 199.0 -> 0.00 mm
- net /D1: track 189.2 -> 0.00 mm
- net /D0: track 186.5 -> 0.00 mm
- net /A0: track 162.1 -> 0.00 mm
- net Net-(IC1-~{CLK}): track 157.0 -> 0.00 mm, vias 1 -> 0
- net Net-(U2-~{CS}): track 145.5 -> 0.00 mm
- net ~{RD}: track 144.5 -> 0.00 mm
- net ~{MREQ}: track 143.3 -> 0.00 mm
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Other:
- board size 154.9 x 129.5 mm -> 152.4 x 129.5 mm

Commit message: Added text
Other:
- board text added: "Itch.io https://adrianpilko.itch.io Github https://github.com/AdrianPilko Youtube @byteforever7829"
Changed lines of the file:
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@@
   (gr_line (start 55.88 162.56) (end 58.42 162.56)
     (stroke (width 0.1) (type default)) (layer "Edge.Cuts"))
+  (gr_text "Itch.io  https://adrianpilko.itch.io\nGithub   https://github.com/AdrianPilko\nYoutube  @byteforever7829" (at 165.1 40.64) (layer "Edge.Cuts")
+    (effects (font (size 1 1) (thickness 0.15)) (justify left bottom))
+  )
   (segment (start 53.34 40.64) (end 58.42 40.64) (width 0.25) (layer "F.Cu") (net 1))
   (segment (start 58.42 35.56) (end 58.42 40.64) (width 0.25) (layer "B.Cu") (net 1))

Commit message: autorouted
Routing:
- net Z80_PWRCAP: track 15.2 -> 537.7 mm, vias 0 -> 1
- net +5V: track 0.00 -> 455.6 mm, vias 0 -> 1
- net /D1: track 0.00 -> 275.2 mm
- net /D5: track 0.00 -> 262.0 mm, vias 0 -> 1
- net /D4: track 0.00 -> 246.5 mm, vias 0 -> 1
- net /D2: track 0.00 -> 244.0 mm, vias 0 -> 2
- net /D3: track 0.00 -> 239.5 mm
- net /D7: track 0.00 -> 235.5 mm, vias 0 -> 1
- net /D6: track 0.00 -> 222.1 mm, vias 0 -> 1
- net /D0: track 0.00 -> 215.9 mm, vias 0 -> 1
- net Net-(IC1-~{RESET}): track 0.00 -> 208.9 mm
- net ~{RD}: track 0.00 -> 165.8 mm
- net ~{MREQ}: track 0.00 -> 154.1 mm, vias 0 -> 1
- net /A0: track 0.00 -> 145.2 mm, vias 0 -> 1
- net /A15: track 0.00 -> 142.0 mm
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